File: RoboFest_IGVC_Circuit/mcu_esp32.kicad_sch (KiCad schematic)
At the start: 0 parts

Commit message: updated diagram
Parts:
- added U4: STM32F446RETx, Package_QFP:LQFP-64_10x10mm_P0.5mm, symbol MCU_ST_STM32F4:STM32F446RETx
Connections:
- new net 3V3: U4.19 (VDD)
- new net ENC1_A: U4.50 (PA15)
- new net ENC1_B: U4.15 (PA1)
- new net ENC2_A: U4.22 (PA6)
- new net ENC2_B: U4.23 (PA7)
- new net ENC3_A: U4.58 (PB6)
- new net ENC3_B: U4.59 (PB7)
- new net ENC4_A: U4.37 (PC6)
- new net ENC4_B: U4.38 (PC7)
- new net ESTOP_SENSE: U4.51 (PC10)
- new net GND: U4.18 (VSS), U4.31 (VSS), U4.47 (VSS), U4.63 (VSS)
- new net I2C1_SCL: U4.61 (PB8)
- new net I2C1_SDA: U4.62 (PB9)
- new net M1_DIR: U4.8 (PC0)
- new net M1_PWM: U4.41 (PA8)
- new net M2_DIR: U4.9 (PC1)
- new net M2_PWM: U4.42 (PA9)
- new net M3_DIR: U4.10 (PC2)
- new net M3_PWM: U4.43 (PA10)
- new net M4_DIR: U4.11 (PC3)
- new net M4_PWM: U4.44 (PA11)
- new net SERVO1_PWM: U4.35 (PB14)
- new net SERVO2_PWM: U4.36 (PB15)
- new net SERVO3_PWM: U4.14 (PA0)
- new net STATUS_LED: U4.21 (PA5)
- new net TOF1_XSHUT: U4.24 (PC4)
- new net TOF2_XSHUT: U4.25 (PC5)
- new net TOF3_XSHUT: U4.26 (PB0)
- new net TOF4_XSHUT: U4.27 (PB1)
- new net USART2_RX: U4.17 (PA3)
- new net USART2_TX: U4.16 (PA2)
Other:
- note added: "MCU STM32 Nucleo F446RETx Module"

Commit message: updated diagram
Parts:
- added C1: 4.7 µF low-ESR ceramic cap, symbol Device:C
- added C2: 100nF, symbol Device:C
- added R3: 10k, symbol Device:R
Connections:
- net GND: now also C1.1, C2.1, R3.1
- net at U4.30 (VCAP_1): now also C1.2
- net SERVO4_PWM: now reaches U4.34 (PB13)
- net at U4.60 (BOOT0): now also R3.2
- net at U4.7 (NRST): now also C2.2
- no-connect marks 0 -> 26

Commit message: added cad files
Changed lines of the file:
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@@
+	)
+	(junction
+		(at 147.32 46.99)
+		(diameter 0)
+		(color 0 0 0 0)
 	)
 	(junction
@@
 	(wire
 		(pts
+			(xy 147.32 46.99) (xy 147.32 50.8)
+		)
+		(stroke
+			(width 0)
+			(type default)
+		)
+	)
+	(wire
+		(pts
 			(xy 125.73 63.5) (xy 129.54 63.5)
 		)
@@
 	(wire
 		(pts
-			(xy 147.32 44.45) (xy 147.32 50.8)
+			(xy 147.32 44.45) (xy 147.32 46.99)
 		)
 		(stroke
@@
 		)
 	)
+	(symbol
+		(lib_id "power:PWR_FLAG")
+		(at 147.32 46.99 270)
+		(unit 1)
+		(body_style 1)
+		(exclude_from_sim no)
+		(in_bom yes)
+		(on_board yes)
+		(in_pos_files yes)
+		(dnp no)
+		(fields_autoplaced yes)
+		(property "Reference" "#FLG06"
+			(at 149.225 46.99 0)
+			(hide yes)
+			(show_name no)
+			(do_not_autoplace no)
+			(effects
+				(font
+					(size 1.27 1.27)
+				)
+			)
+		)
+		(property "Value" "PWR_FLAG"
+			(at 151.13 46.9899 90)
+			(show_name no)
+			(do_not_autoplace no)
+			(effects
+				(font
+					(size 1.27 1.27)
+				)
+				(justify left)
+			)
+		)
+		(property "Footprint" ""
+			(at 147.32 46.99 0)
+			(hide yes)
+			(show_name no)
+			(do_not_autoplace no)
+			(effects
+				(font
+					(size 1.27 1.27)
+				)
+			)
+		)
+		(property "Datasheet" ""
+			(at 147.32 46.99 0)
+			(hide yes)
+			(show_name no)
+			(do_not_autoplace no)
+			(effects
+				(font
+					(size 1.27 1.27)
+				)
+			)
+		)
+		(property "Description" "Special symbol for telling ERC where power comes from"
+			(at 147.32 46.99 0)
+			(hide yes)
+			(show_name no)
+			(do_not_autoplace no)
+			(effects
+				(font
+					(size 1.27 1.27)
+				)
+			)
+		)
+		(pin "1"
+		)
+		(instances
+			(project "RoboFest_IGVC_Circuit"
+				(path "/bd507979-6024-412b-bdc6-54c3e4be9cc9/f0428bdc-3c83-4dd4-b381-7b729ef35c11"
+					(reference "#FLG06")
+					(unit 1)
+				)
+			)
+		)
+	)
