File: RoboFest_IGVC_Circuit/motor_drive.kicad_sch (KiCad schematic)
At the start: 0 parts

Commit message: updated diagram
Parts:
- added J10: Encoder 3 RL, symbol Connector_Generic:Conn_01x04
- added J11: Encoder 4 RR, symbol Connector_Generic:Conn_01x04
- added J12: Cytron MDD10A Left, symbol Connector_Generic:Conn_01x06
- added J13: Cytron MDD10A Right, symbol Connector_Generic:Conn_01x06
- added J14, J15: Cytron Output Left, symbol Connector_Generic:Conn_01x04
- added J8: Encoder 1 FL, symbol Connector_Generic:Conn_01x04
- added J9: Encoder 2 FR, symbol Connector_Generic:Conn_01x04
- added M1: 12V DC gear motors FL, symbol Motor:Motor_DC
- added M2: 12V DC gear motors FR, symbol Motor:Motor_DC
- added M3: 12V DC gear motors RL, symbol Motor:Motor_DC
- added M4: 12V DC gear motors RR, symbol Motor:Motor_DC
Connections:
- new net: J14.4 (Pin_4), M1.1 (+)
- new net: J14.3 (Pin_3), M1.2 (-)
- new net: J14.2 (Pin_2), M3.1 (+)
- new net: J14.1 (Pin_1), M3.2 (-)
- new net: J15.2 (Pin_2), M4.1 (+)
- new net: J15.1 (Pin_1), M4.2 (-)
- new net: J15.4 (Pin_4), M2.1 (+)
- new net: J15.3 (Pin_3), M2.2 (-)
- new net 5V_LOGIC: J10.1 (VCC), J8.1 (VCC), J9.1 (VCC)
- new net ENC1_A: J8.3 (CH_A)
- new net ENC1_B: J8.4 (CH_B)
- new net ENC2_A: J9.3 (CH_A)
- new net ENC2_B: J9.4 (CH_B)
- new net ENC3_A: J10.3 (CH_A)
- new net ENC3_B: J10.4 (CH_B)
- new net ENC4_A: J11.3 (CH_A)
- new net ENC4_B: J11.4 (CH_B)
- new net GND: J10.2 (GND), J11.2 (GND), J12.2 (Pin_2), J13.2 (Pin_2), J8.2 (GND), J9.2 (GND)
- new net M1_DIR: J12.4 (Pin_4)
- new net M1_PWM: J12.3 (Pin_3)
- new net M2_DIR: J12.6 (Pin_6)
- new net M2_PWM: J12.5 (Pin_5)
- new net M3_DIR: J13.4 (Pin_4)
- new net M3_PWM: J13.3 (Pin_3)
- new net M4_DIR: J13.6 (Pin_6)
- new net M4_PWM: J13.5 (Pin_5)
- new net MOTOR_12V: J12.1 (Pin_1), J13.1 (Pin_1)
Other:
- note added: "14AWG"
- note added: "16-18AWG Silicone"
- note added: "22-24AWG Twisted Pair"
- note added: "Encoder Module"
- note added: "FL"
- note added: "FR"
- note added: "Motor + driver Module"
- note added: "RL"
- note added: "RR"

Commit message: added cad files
Connections:
- net 5V_LOGIC: now also J11.1 (VCC)
Changed lines of the file:
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@@
 	)
 	(label "5V_LOGIC"
-		(at 187.96 124.46 180)
+		(at 189.23 124.46 180)
 		(effects
 			(font
