File: RoboFest_IGVC_Circuit/sbc_interconnect.kicad_sch (KiCad schematic)
At the start: 0 parts

Commit message: updated diagram
Parts:
- added J7: Raspberry_Pi_2_3, symbol Connector:Raspberry_Pi_2_3
Connections:
- new net: J7.14 (GND), J7.20 (GND), J7.25 (GND), J7.30 (GND), J7.34 (GND), J7.39 (GND), J7.6 (GND), J7.9 (GND)
- new net 5V_PI: J7.2 (5V), J7.4 (5V)
- new net GND: J7.1 (3V3), J7.17 (3V3)

Commit message: updated diagram
Connections:
- net GND: now also J7.14 (GND), J7.20 (GND), J7.25 (GND), J7.30 (GND), J7.34 (GND), J7.39 (GND), J7.6 (GND), J7.9 (GND); no longer J7.1 (3V3), J7.17 (3V3)
- net USART_TX: now reaches J7.10 (GPIO15/RXD)
- net USART_RX: now reaches J7.8 (GPIO14/TXD)
- new net: J7.1 (3V3), J7.17 (3V3)
- no-connect marks 0 -> 27
Changed lines of the file:
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@@
 		(comment 1 "Nirma University")
 	)
+	(no_connect
+		(at 115.57 95.25)
+	)
+	(no_connect
+		(at 156.21 102.87)
+	)
+	(no_connect
+		(at 156.21 59.69)
+	)
+	(no_connect
+		(at 115.57 97.79)
+	)
+	(no_connect
+		(at 156.21 74.93)
+	)
+	(no_connect
+		(at 156.21 62.23)
+	)
+	(no_connect
+		(at 156.21 69.85)
+	)
+	(no_connect
+		(at 156.21 77.47)
+	)
+	(no_connect
+		(at 115.57 69.85)
+	)
+	(no_connect
+		(at 156.21 90.17)
+	)
+	(no_connect
+		(at 115.57 100.33)
+	)
+	(no_connect
+		(at 156.21 87.63)
+	)
+	(no_connect
+		(at 156.21 85.09)
+	)
+	(no_connect
+		(at 140.97 43.18)
+	)
+	(no_connect
+		(at 156.21 80.01)
+	)
+	(no_connect
+		(at 115.57 72.39)
+	)
+	(no_connect
+		(at 156.21 95.25)
+	)
+	(no_connect
+		(at 115.57 90.17)
+	)
+	(no_connect
+		(at 115.57 67.31)
+	)
+	(no_connect
+		(at 156.21 92.71)
+	)
+	(no_connect
+		(at 115.57 77.47)
+	)
+	(no_connect
+		(at 156.21 100.33)
+	)
+	(no_connect
+		(at 156.21 67.31)
+	)
+	(no_connect
+		(at 115.57 92.71)
+	)
+	(no_connect
+		(at 115.57 80.01)
+	)
+	(no_connect
+		(at 115.57 82.55)
+	)
+	(no_connect
+		(at 115.57 87.63)
+	)
+	(wire
+		(pts
+			(xy 110.49 59.69) (xy 115.57 59.69)
+		)
+		(stroke
+			(width 0)
+			(type default)
+		)
+	)
+	(wire
+		(pts
+			(xy 135.89 115.57) (xy 135.89 119.38)
+		)
+		(stroke
+			(width 0)
+			(type default)
+		)
+	)
+	(wire
+		(pts
+			(xy 110.49 62.23) (xy 115.57 62.23)
+		)
+		(stroke
+			(width 0)
+			(type default)
+		)
+	)
 	(wire
 		(pts
@@
 			(width 0)
 			(type default)
+		)
+	)
+	(label "USART_RX"
+		(at 110.49 59.69 180)
+		(effects
+			(font
+				(size 1.27 1.27)
+			)
+			(justify right bottom)
+		)
+	)
+	(label "USART_TX"
+		(at 110.49 62.23 180)
+		(effects
+			(font
+				(size 1.27 1.27)
+			)
+			(justify right bottom)
 		)
 	)
@@
 	(symbol
 		(lib_id "power:GND")
-		(at 140.97 43.18 180)
+		(at 135.89 119.38 0)
 		(unit 1)
 		(body_style 1)
@@
 		(fields_autoplaced yes)
 		(property "Reference" "#PWR010"
-			(at 140.97 36.83 0)
+			(at 135.89 125.73 0)
 			(hide yes)
 			(show_name no)
@@
 		)
 		(property "Value" "GND"
-			(at 140.97 38.1 0)
+			(at 135.89 124.46 0)
 			(show_name no)
 			(do_not_autoplace no)
@@
 		)
 		(property "Footprint" ""
-			(at 140.97 43.18 0)
+			(at 135.89 119.38 0)
 			(hide yes)
 			(show_name no)
@@
 		)
 		(property "Datasheet" ""
-			(at 140.97 43.18 0)
+			(at 135.89 119.38 0)
 			(hide yes)
 			(show_name no)
@@
 		)
 		(property "Description" "Power symbol creates a global label with name \"GND\" , ground"
-			(at 140.97 43.18 0)
-			(hide yes)
-			(show_name no)
+			(at 135.89 119.38 0)
+			(hide yes)
+			(show_name no)

Commit message: added cad files
Changed lines of the file:
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@@
 		(comment 1 "Nirma University")
 	)
+	(junction
+		(at 130.81 47.027)
+		(diameter 0)
+		(color 0 0 0 0)
+	)
 	(no_connect
 		(at 115.57 95.25)
@@
 	(wire
 		(pts
+			(xy 130.81 47.027) (xy 130.81 49.53)
+		)
+		(stroke
+			(width 0)
+			(type default)
+		)
+	)
+	(wire
+		(pts
 			(xy 135.89 115.57) (xy 135.89 119.38)
 		)
@@
 	(wire
 		(pts
-			(xy 130.81 43.18) (xy 130.81 49.53)
+			(xy 130.81 43.18) (xy 130.81 47.027)
 		)
 		(stroke
@@
 		)
 	)
+	(symbol
+		(lib_id "power:PWR_FLAG")
+		(at 130.81 47.027 90)
+		(unit 1)
+		(body_style 1)
+		(exclude_from_sim no)
+		(in_bom yes)
+		(on_board yes)
+		(in_pos_files yes)
+		(dnp no)
+		(fields_autoplaced yes)
+		(property "Reference" "#FLG014"
+			(at 128.905 47.027 0)
+			(hide yes)
+			(show_name no)
+			(do_not_autoplace no)
+			(effects
+				(font
+					(size 1.27 1.27)
+				)
+			)
+		)
+		(property "Value" "PWR_FLAG"
+			(at 127 47.0269 90)
+			(show_name no)
+			(do_not_autoplace no)
+			(effects
+				(font
+					(size 1.27 1.27)
+				)
+				(justify left)
+			)
+		)
+		(property "Footprint" ""
+			(at 130.81 47.027 0)
+			(hide yes)
+			(show_name no)
+			(do_not_autoplace no)
+			(effects
+				(font
+					(size 1.27 1.27)
+				)
+			)
+		)
+		(property "Datasheet" ""
+			(at 130.81 47.027 0)
+			(hide yes)
+			(show_name no)
+			(do_not_autoplace no)
+			(effects
+				(font
+					(size 1.27 1.27)
+				)
+			)
+		)
+		(property "Description" "Special symbol for telling ERC where power comes from"
+			(at 130.81 47.027 0)
+			(hide yes)
+			(show_name no)
+			(do_not_autoplace no)
+			(effects
+				(font
+					(size 1.27 1.27)
+				)
+			)
+		)
+		(pin "1"
+		)
+		(instances
+			(project "RoboFest_IGVC_Circuit"
+				(path "/bd507979-6024-412b-bdc6-54c3e4be9cc9/05a854fa-321e-48c8-b532-78f2b336a09a"
+					(reference "#FLG014")
+					(unit 1)
+				)
+			)
+		)
+	)
