File: RoboFest_IGVC_Circuit/sensors.kicad_sch (KiCad schematic)
At the start: 0 parts

Commit message: added STM32 pinout and report and code
Parts:
- added U1: VL53L1CXV0FY1, Sensor_Distance:ST_VL53L1x, symbol Sensor_Distance:VL53L1CXV0FY1
- added U2: 2472, 2472:MODULE_2472, symbol VL53L1X:2472
Connections:
- new net: U1.12 (GND), U1.3 (GND), U1.4 (GND), U1.6 (GND)

Commit message: updated diagram
Parts:
- removed U1: VL53L1CXV0FY1, Sensor_Distance:ST_VL53L1x, symbol Sensor_Distance:VL53L1CXV0FY1
- removed U2: 2472, 2472:MODULE_2472, symbol VL53L1X:2472

Commit message: added cad files
Parts:
- added R4: 10k, symbol Device:R
- added U1: BNO055, 2472:MODULE_2472, symbol BNO055:2472
- added U2: VL53L1X 1, Sensor_Distance:ST_VL53L1x, symbol Sensor_Distance:VL53L1CXV0FY1
- added U6: VL53L1X 2, Sensor_Distance:ST_VL53L1x, symbol Sensor_Distance:VL53L1CXV0FY1
- added U7: VL53L1X 3, Sensor_Distance:ST_VL53L1x, symbol Sensor_Distance:VL53L1CXV0FY1
- added U8: VL53L1X 4, Sensor_Distance:ST_VL53L1x, symbol Sensor_Distance:VL53L1CXV0FY1
Connections:
- new net: R4.2, U1.6 (RST)
- new net 3V3: R4.1
- new net 5V_LOGIC: U1.1 (VIN), U2.1 (AVDDVCSEL), U2.11 (AVDD), U6.1 (AVDDVCSEL), U6.11 (AVDD), U7.1 (AVDDVCSEL), U7.11 (AVDD), U8.1 (AVDDVCSEL), U8.11 (AVDD)
- new net GND: U1.3 (GND), U1.7 (ADR), U2.12 (GND), U2.2 (AVSSVCSEL), U2.3 (GND), U2.4 (GND), U2.6 (GND), U6.12 (GND), U6.2 (AVSSVCSEL), U6.3 (GND), U6.4 (GND), U6.6 (GND), U7.12 (GND), U7.2 (AVSSVCSEL), U7.3 (GND), U7.4 (GND), U7.6 (GND), U8.12 (GND), U8.2 (AVSSVCSEL), U8.3 (GND), U8.4 (GND), U8.6 (GND)
- new net I2C1_SCL: U1.5 (SCL), U2.10 (SCL), U6.10 (SCL), U7.10 (SCL), U8.10 (SCL)
- new net I2C1_SDA: U1.4 (SDA), U2.9 (SDA), U6.9 (SDA), U7.9 (SDA), U8.9 (SDA)
- new net TOF1_XSHUT: U2.5 (XSHUT)
- new net TOF2_XSHUT: U6.5 (XSHUT)
- new net TOF3_XSHUT: U7.5 (XSHUT)
- new net TOF4_XSHUT: U8.5 (XSHUT)
- no-connect marks 0 -> 8
