File: RoboFest_IGVC_Circuit/suspension_actuation.kicad_sch (KiCad schematic)
At the start: 0 parts

Commit message: added cad files
Parts:
- added M5, M6, M7, M8: Motor_Servo, symbol Motor:Motor_Servo
Connections:
- new net 5V_SERVO: M5.2 (+), M6.2 (+), M7.2 (+), M8.2 (+)
- new net GND: M5.3 (-), M6.3 (-), M7.3 (-), M8.3 (-)
- new net SERVO1_PWM: M5.1 (PWM)
- new net SERVO2_PWM: M6.1 (PWM)
- new net SERVO3_PWM: M7.1 (PWM)
- new net SERVO4_PWM: M8.1 (PWM)
